Commit message: Imported upstream version '1.1.7' of 'upstream'

File: abb_irb2400_support/urdf/irb2400.urdf (robot description, URDF)
Before this commit: robot abb_irb2400, 8 links, 7 joints
Links:
- added link base
Joints:
- added joint base_link-base: type fixed, parent base_link, child base, origin xyz=0 0 0 rpy=0 0 0
- joint joint_6-tool0: origin xyz=0 0 0 rpy=0 0 0 -> xyz=0 0 0 rpy=0 1.57079632679 0

File: abb_irb2400_support/urdf/irb2400_macro.xacro (robot description, xacro)
@@ -127,6 +127,4 @@
         <axis xyz="0 0 1"/>
         <limit lower="-3.1416" upper="3.1416" effort="0" velocity="2.618"/>
-        <calibration rising="0" falling="0"/>
-        <dynamics damping="0" friction="0"/>
     </joint>
     <joint name="${prefix}joint_2" type="revolute">
@@ -136,6 +134,4 @@
         <axis xyz="0 1 0"/>
         <limit lower="-1.7453" upper="1.9199" effort="0" velocity="2.618"/>
-        <calibration rising="0" falling="0"/>
-        <dynamics damping="0" friction="0"/>
     </joint>
     <joint name="${prefix}joint_3" type="revolute">
@@ -145,6 +141,4 @@
         <axis xyz="0 1 0"/>
         <limit lower="-1.0472" upper="1.1345" effort="0" velocity="2.618"/>
-        <calibration rising="0" falling="0"/>
-        <dynamics damping="0" friction="0"/>
     </joint>
     <joint name="${prefix}joint_4" type="revolute">
@@ -154,6 +148,4 @@
         <axis xyz="1 0 0"/>
         <limit lower="-3.49" upper="3.49" effort="0" velocity="6.2832"/>
-        <calibration rising="0" falling="0"/>
-        <dynamics damping="0" friction="0"/>
     </joint>
     <joint name="${prefix}joint_5" type="revolute">
@@ -163,6 +155,4 @@
         <axis xyz="0 1 0"/>
         <limit lower="-2.0944" upper="2.0944" effort="0" velocity="6.2832"/>
-        <calibration rising="0" falling="0"/>
-        <dynamics damping="0" friction="0"/>
     </joint>
     <joint name="${prefix}joint_6" type="revolute">
@@ -172,13 +162,18 @@
         <axis xyz="1 0 0"/>
         <limit lower="-6.9813" upper="6.9813" effort="0" velocity="7.854"/>
-        <calibration rising="0" falling="0"/>
-        <dynamics damping="0" friction="0"/>
     </joint>
     <joint name="${prefix}joint_6-tool0" type="fixed">
         <parent link="${prefix}link_6"/>
         <child link="${prefix}tool0"/>
-        <origin xyz="0 0 0" rpy="0 0 0"/>
+        <origin xyz="0 0 0" rpy="0 1.57079632679 0"/>
     </joint>
     <!-- end of joint list -->
+    <!-- ROS base_link to ABB World Coordinates transform -->
+    <link name="${prefix}base" />
+    <joint name="${prefix}base_link-base" type="fixed">
+        <origin xyz="0 0 0" rpy="0 0 0"/>
+        <parent link="${prefix}base_link"/>
+        <child link="${prefix}base"/>
+    </joint>
 </xacro:macro>
 </robot>

File: abb_irb5400_support/urdf/irb5400.urdf (robot description, URDF)
Before this commit: robot abb_irb5400, 9 links, 8 joints
Links:
- added link base
Joints:
- added joint base_link-base: type fixed, parent base_link, child base, origin xyz=0 0 0 rpy=0 0 0
- joint joint_6-tool0: origin xyz=0.0672 0 -0.0470 rpy=0.0 0.6109 0.0 -> xyz=0 0 0 rpy=0 1.57079632679 0

File: abb_irb5400_support/urdf/irb5400_macro.xacro (robot description, xacro)
@@ -177,7 +177,14 @@
         <parent link="${prefix}link_6"/>
         <child link="${prefix}tool0"/>
-        <origin xyz="0.0672 0 -0.0470" rpy="0.0 0.6109 0.0"/>
+        <origin xyz="0 0 0" rpy="0 1.57079632679 0"/>
     </joint>
     <!-- end of joint list -->
+    <!-- ROS base_link to ABB World Coordinates transform -->
+    <link name="${prefix}base" />
+    <joint name="${prefix}base_link-base" type="fixed">
+        <origin xyz="0 0 0" rpy="0 0 0"/>
+        <parent link="${prefix}base_link"/>
+        <child link="${prefix}base"/>
+    </joint>
 </xacro:macro>
 </robot>

File: abb_irb6600_support/urdf/irb6640.urdf (robot description, URDF)
Before this commit: robot abb_irb6640, 10 links, 9 joints
Links:
- added link base
Joints:
- added joint base_link-base: type fixed, parent base_link, child base, origin xyz=0 0 0 rpy=0 0 0
- joint joint_6-tool0: axis 1 0 0 -> (none); origin xyz=.055 0 0  rpy=0 0 0 -> xyz=.055 0 0 rpy=0 1.57079632679 0

File: abb_irb6600_support/urdf/irb6640_macro.xacro (robot description, xacro)
@@ -179,9 +179,8 @@
         <limit effort="0" lower="-6.283" upper="6.283" velocity="3.3161"/>
     </joint>
-    <joint type="fixed" name="joint_6-tool0">
-        <origin xyz=".055 0 0 " rpy="0 0 0"/>
-        <axis xyz="1 0 0"/>
+    <joint type="fixed" name="${prefix}joint_6-tool0">
         <parent link="${prefix}link_6"/>
         <child link="${prefix}tool0"/>
+        <origin xyz=".055 0 0" rpy="0 1.57079632679 0"/>
     </joint>
     <joint type="fixed" name="${prefix}joint_cylinder">
@@ -200,4 +199,11 @@
     </joint>
     <!-- end of joint list -->
+    <!-- ROS base_link to ABB World Coordinates transform -->
+    <link name="${prefix}base" />
+    <joint name="${prefix}base_link-base" type="fixed">
+        <origin xyz="0 0 0" rpy="0 0 0"/>
+        <parent link="${prefix}base_link"/>
+        <child link="${prefix}base"/>
+    </joint>
 </xacro:macro>
 </robot>
